File: QuadCAN-FD.kicad_pcb (KiCad board)
At the start: 2 copper layers, 25.4 x 53.3 mm, 48 parts, among them J1 Raspberry_Pi_2_3, J2 Conn_02x04_Odd_Even, U1 MCP2517FD-xSL, U2 MCP2517FD-xSL, U3 MCP2517FD-xSL, U4 MCP2517FD-xSL, U5 TJA1049T-3, U6 TJA1049T-3, U7 TJA1049T-3, U8 TJA1049T-3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

Commit message: Imported to KiCAD 8
Other:
- net class Default removed
- net class pwr removed
